File: sis5351a GPS controlled time base.kicad_sch (KiCad schematic)
At the start: 47 parts, among them J1 USB_B_Micro, J2 Conn_01x05_Pin, J3 Conn_01x04_Pin, J4 Conn_02x03_Odd_Even, J5 Conn_01x12_Pin, J6 Conn_Coaxial, J7 Conn_Coaxial, Q1 BSS138, Q2 BSS138, U1 Si5351A-B-GT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

Commit message: Fault in I2C level converter
Parts:
- removed R7, R8: 1K, Resistor_SMD:R_0805_2012Metric_Pad1.20x1.40mm_HandSolder, symbol Device:R
- Y1: footprint Crystal:Crystal_SMD_Abracon_ABM8AIG-4Pin_3.2x2.5mm -> Crystal:Crystal_SMD_3225-4Pin_3.2x2.5mm_HandSoldering
Connections:
- net +3V3: now also R1.1, R2.1; no longer R3.1, R4.1
- net +5V: now also R3.1, R4.1; no longer R1.1, R2.1
- net SCL3: now also Q1.2 (S), R2.2; no longer Q1.3 (D), R3.2
- net SCL5: now also Q1.3 (D), R3.2; no longer Q1.2 (S), R2.2
- net SDA3: now also Q2.2 (S), R1.2; no longer Q2.3 (D), R4.2
- net SDA5: now also Q2.3 (D), R4.2; no longer Q2.2 (S), R1.2
- net USB_RXD: now also U5.1 (TXD)
- net USB_TXD: now also U5.5 (RXD)
Changed lines of the file:
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@@
 	(wire
 		(pts
-			(xy 250.19 59.69) (xy 250.19 62.23)
-		)
-		(stroke
-			(width 0)
-			(type default)
-		)
-	)
-	(wire
-		(pts
 			(xy 40.64 140.97) (xy 35.56 140.97)
 		)
@@
 	(wire
 		(pts
-			(xy 242.57 59.69) (xy 242.57 62.23)
-		)
-		(stroke
-			(width 0)
-			(type default)
-		)
-	)
-	(wire
-		(pts
 			(xy 200.66 106.68) (xy 198.12 106.68)
 		)
@@
 	(wire
 		(pts
-			(xy 242.57 71.12) (xy 242.57 69.85)
+			(xy 242.57 59.69) (xy 242.57 71.12)
 		)
 		(stroke
@@
 	(wire
 		(pts
-			(xy 250.19 73.66) (xy 250.19 69.85)
+			(xy 250.19 59.69) (xy 250.19 73.66)
 		)
 		(stroke
@@
 	(global_label "SCL5"
 		(shape input)
-		(at 86.36 41.91 180)
+		(at 135.89 41.91 0)
 		(fields_autoplaced yes)
 		(effects
@@
 				(size 1.27 1.27)
 			)
-			(justify right)
+			(justify left)
 		)
 		(property "Intersheetrefs" "${INTERSHEET_REFS}"
-			(at 78.6577 41.91 0)
+			(at 143.5923 41.91 0)
 			(effects
 				(font
 					(size 1.27 1.27)
 				)
-				(justify right)
+				(justify left)
 				(hide yes)
 			)
@@
 	(global_label "SCL3"
 		(shape output)
-		(at 135.89 41.91 0)
+		(at 86.36 41.91 180)
 		(fields_autoplaced yes)
 		(effects
@@
 				(size 1.27 1.27)
 			)
-			(justify left)
+			(justify right)
 		)
 		(property "Intersheetrefs" "${INTERSHEET_REFS}"
-			(at 143.5923 41.91 0)
+			(at 78.6577 41.91 0)
 			(effects
 				(font
 					(size 1.27 1.27)
 				)
-				(justify left)
+				(justify right)
 				(hide yes)
 			)
@@
 	(global_label "SDA3"
 		(shape output)
-		(at 135.89 29.21 0)
+		(at 86.36 29.21 180)
 		(fields_autoplaced yes)
 		(effects
@@
 				(size 1.27 1.27)
 			)
-			(justify left)
+			(justify right)
 		)
 		(property "Intersheetrefs" "${INTERSHEET_REFS}"
-			(at 143.6528 29.21 0)
+			(at 78.5972 29.21 0)
 			(effects
 				(font
 					(size 1.27 1.27)
 				)
-				(justify left)
+				(justify right)
 				(hide yes)
 			)
@@
 	(global_label "SDA5"
 		(shape input)
-		(at 86.36 29.21 180)
+		(at 135.89 29.21 0)
 		(fields_autoplaced yes)
 		(effects
@@
 				(size 1.27 1.27)
 			)
-			(justify right)
+			(justify left)
 		)
 		(property "Intersheetrefs" "${INTERSHEET_REFS}"
-			(at 78.5972 29.21 0)
+			(at 143.6528 29.21 0)
 			(effects
 				(font
 					(size 1.27 1.27)
 				)
-				(justify right)
+				(justify left)
 				(hide yes)
 			)
@@
 	(symbol
 		(lib_id "power:+5V")
-		(at 95.25 20.32 0)
+		(at 124.46 20.32 0)
 		(unit 1)
 		(exclude_from_sim no)
@@
 		(fields_autoplaced yes)
 		(property "Reference" "#PWR012"
-			(at 95.25 24.13 0)
+			(at 124.46 24.13 0)
 			(effects
 				(font
@@
 		)
 		(property "Value" "+5V"
-			(at 95.25 15.24 0)
+			(at 124.46 15.24 0)
 			(effects
 				(font
@@
 		)
 		(property "Footprint" ""
-			(at 95.25 20.32 0)
+			(at 124.46 20.32 0)
 			(effects
 				(font
@@
 		)
 		(property "Datasheet" ""
-			(at 95.25 20.32 0)
+			(at 124.46 20.32 0)
 			(effects
 				(font
@@
 		)
 		(property "Description" ""
-			(at 95.25 20.32 0)
+			(at 124.46 20.32 0)
 			(effects
 				(font
@@
 	(symbol
 		(lib_id "power:+3V3")
-		(at 132.08 20.32 0)
+		(at 102.87 20.32 0)
 		(unit 1)
 		(exclude_from_sim no)
@@
 		(fields_autoplaced yes)
 		(property "Reference" "#PWR015"
-			(at 132.08 24.13 0)
+			(at 102.87 24.13 0)
 			(effects
 				(font
@@
 		)
 		(property "Value" "+3V3"
-			(at 132.08 15.24 0)
+			(at 102.87 15.24 0)
 			(effects
 				(font
@@
 		)
 		(property "Footprint" ""
-			(at 132.08 20.32 0)
+			(at 102.87 20.32 0)
 			(effects
 				(font
@@
 		)
 		(property "Datasheet" ""
-			(at 132.08 20.32 0)
+			(at 102.87 20.32 0)
 			(effects
 				(font
@@
 		)
 		(property "Description" ""
-			(at 132.08 20.32 0)
+			(at 102.87 20.32 0)
 			(effects
 				(font
@@
 	(symbol
 		(lib_id "power:+5V")
-		(at 102.87 20.32 0)
+		(at 132.08 20.32 0)
 		(unit 1)
 		(exclude_from_sim no)
@@
 		(fields_autoplaced yes)
 		(property "Reference" "#PWR013"
-			(at 102.87 24.13 0)
+			(at 132.08 24.13 0)
 			(effects
 				(font
@@
 		)
 		(property "Value" "+5V"
-			(at 102.87 15.24 0)
+			(at 132.08 15.24 0)
 			(effects
 				(font
@@
 		)
 		(property "Footprint" ""
-			(at 102.87 20.32 0)
+			(at 132.08 20.32 0)
 			(effects
 				(font
@@
 		)
 		(property "Datasheet" ""
-			(at 102.87 20.32 0)
+			(at 132.08 20.32 0)
 			(effects
 				(font
@@
 		)
 		(property "Description" ""
-			(at 102.87 20.32 0)
+			(at 132.08 20.32 0)
 			(effects
 				(font
@@
 	)
 	(symbol
-		(lib_id "Device:R")
-		(at 250.19 66.04 0)
-		(unit 1)
-		(exclude_from_sim no)
-		(in_bom yes)
-		(on_board yes)
-		(dnp no)
-		(fields_autoplaced yes)
-		(property "Reference" "R8"
-			(at 252.73 64.77 0)
-			(effects
-				(font
-					(size 1.27 1.27)
-				)
-				(justify left)
-			)
-		)
-		(property "Value" "1K"
-			(at 252.73 67.31 0)
-			(effects
-				(font
-					(size 1.27 1.27)
-				)
-				(justify left)
-			)
-		)
-		(property "Footprint" "Resistor_SMD:R_0805_2012Metric_Pad1.20x1.40mm_HandSolder"
-			(at 248.412 66.04 90)
-			(effects
-				(font
-					(size 1.27 1.27)
-				)
-				(hide yes)
-			)
-		)
-		(property "Datasheet" "~"
-			(at 250.19 66.04 0)
-			(effects
-				(font
-					(size 1.27 1.27)
-				)
-				(hide yes)
-			)
-		)
-		(property "Description" ""
-			(at 250.19 66.04 0)
-			(effects
-				(font
-					(size 1.27 1.27)
-				)
-				(hide yes)
-			)
-		)
-		(pin "1"
-		)
-		(pin "2"
-		)
-		(instances
-			(project "sis5351a GPS controlled time base"
-				(path "/3e92bbdf-4ead-4bfe-9d54-982f224f75c6"
-					(reference "R8")
-					(unit 1)
-				)
-			)
-		)
-	)
-	(symbol
 		(lib_id "Device:C")
 		(at 90.17 143.51 180)
@@
 	(symbol
 		(lib_id "power:+3V3")
-		(at 124.46 20.32 0)
+		(at 95.25 20.32 0)
 		(unit 1)
 		(exclude_from_sim no)
@@
 		(fields_autoplaced yes)
 		(property "Reference" "#PWR014"
-			(at 124.46 24.13 0)
+			(at 95.25 24.13 0)
 			(effects
 				(font
@@
 		)
 		(property "Value" "+3V3"
-			(at 124.46 15.24 0)
+			(at 95.25 15.24 0)
 			(effects
 				(font
@@
 		)
 		(property "Footprint" ""
-			(at 124.46 20.32 0)
+			(at 95.25 20.32 0)
 			(effects
 				(font
@@
 		)
 		(property "Datasheet" ""
-			(at 124.46 20.32 0)
+			(at 95.25 20.32 0)
 			(effects
 				(font
@@
 		)
 		(property "Description" ""
-			(at 124.46 20.32 0)
+			(at 95.25 20.32 0)
 			(effects
 				(font
@@
 	)
 	(symbol
-		(lib_id "Device:R")
-		(at 242.57 66.04 0)
-		(unit 1)
-		(exclude_from_sim no)
-		(in_bom yes)
-		(on_board yes)
-		(dnp no)
-		(fields_autoplaced yes)
-		(property "Reference" "R7"
-			(at 245.11 64.77 0)
-			(effects
-				(font
-					(size 1.27 1.27)
-				)
-				(justify left)
-			)
-		)
-		(property "Value" "1K"
-			(at 245.11 67.31 0)
-			(effects
-				(font
-					(size 1.27 1.27)
-				)
-				(justify left)
-			)
-		)
-		(property "Footprint" "Resistor_SMD:R_0805_2012Metric_Pad1.20x1.40mm_HandSolder"
-			(at 240.792 66.04 90)
-			(effects
-				(font
-					(size 1.27 1.27)
-				)
-				(hide yes)
-			)
-		)
-		(property "Datasheet" "~"
-			(at 242.57 66.04 0)
-			(effects
-				(font
-					(size 1.27 1.27)
-				)
-				(hide yes)
-			)
-		)
-		(property "Description" ""
-			(at 242.57 66.04 0)
-			(effects
-				(font
-					(size 1.27 1.27)
-				)
-				(hide yes)
-			)
-		)
-		(pin "1"
-		)
-		(pin "2"
-		)
-		(instances
-			(project "sis5351a GPS controlled time base"
-				(path "/3e92bbdf-4ead-4bfe-9d54-982f224f75c6"
-					(reference "R7")
-					(unit 1)
-				)
-			)
-		)
-	)
-	(symbol
 		(lib_id "Device:C_Polarized")
 		(at 163.83 38.1 0)
@@
 			)
 		)
-		(property "Footprint" "Crystal:Crystal_SMD_Abracon_ABM8AIG-4Pin_3.2x2.5mm"
+		(property "Footprint" "Crystal:Crystal_SMD_3225-4Pin_3.2x2.5mm_HandSoldering"
 			(at 29.21 85.09 0)
 			(effects
